File: 8250 disk interface board.kicad_pcb (KiCad board)
At the start: 2 copper layers, 138 x 30 mm, 14 parts, among them J1 01x14_Servo connector, P1 Conn_01x04, U1 74LS04

Commit message: Sent off to OshPark
Parts:
- R1, R2, R3, R4: footprint Resistor_THT:R_Axial_DIN0207_L6.3mm_D2.5mm_P7.62mm_Horizontal -> Resistor_THT:R_Axial_DIN0204_L3.6mm_D1.6mm_P5.08mm_Horizontal
- moved R4 2.80 mm to (197.1, 111.7)
- moved R3 2.66 mm to (172.0, 111.8)
- moved C3 1.83 mm to (204.4, 107.0)
- moved R1 0.73 mm to (169.6, 106.7)
- moved U1 0.12 mm to (191.0, 106.7)
- moved R2 0.10 mm to (194.8, 106.7)
Routing:
- net Earth: track 37.6 -> 17.5 mm, vias 0 -> 1
- net +5V: track 46.1 -> 42.8 mm
- net Net-(J1-Pin_08): track 16.3 -> 15.4 mm
- net Net-(J1-Pin_12): track 21.9 -> 21.3 mm
Other:
- board text added: "MPI Servo Board For Comodore 8050/8250 Disk Drive PCB #314227-01 JDTucker V 0.1 09/24/23"
- board text added: "P1"
- board text added: "P2"
- board text added: "P3"
- board text added: "P4"
- board text added: "P5"
- board text removed: "MPI Servo Board For Comodore 8250 Disk Drive PCB #314227-01 JDTucker V 0.1 08/12/23"
